File: light sensor basic.brd (EAGLE design)
At the start: 83.2 x 57.8 mm, 1 part

Commit message: Finished
Parts:
- added C2: 0.1uF, rcl:C1206
- added J1: UJ2-MIBH-G-SMT-TR, UJ2-MIBH-G-SMT-TR:CUI_UJ2-MIBH-G-SMT-TR
- added K<LED1: (no value), led:CHIPLED_0805
- added Q1: (no value), semicon-smd-ipc:SOT23
- added R1: 82, rcl:R1206
- added R2: TC33X-2-203E, TC33X-2-203E:TRIM_TC33X-2-203E
- added R3: 150, rcl:R0805
- added TP1, TP2, TP3, TP4: (no value), rcl:R1206
- added U1: VCNT2020, VCNT2020:XDCR_VCNT2020
- moved U$1 106.9 mm to (-106.7, 6.35)
Connections:
- new net GND: C2.1, J1.5, J1.S1, J1.S2, J1.S3, J1.S4, Q1.2, R2.3, TP2.1, TP2.2, U1.4
- new net N$1: R1.2, U1.3
- new net N$2: K<LED1.C, Q1.3
- new net N$3: R2.1, TP1.1, TP1.2, U1.1
- new net N$4: K<LED1.A, R3.1
- new net N$5: Q1.1, R2.2, TP3.1, TP3.2
- new net VCC: C2.2, J1.1, R1.1, R3.2, TP4.1, TP4.2, U1.2
Routing:
- net VCC: track 0.00 -> 119.0 mm
- net GND: track 0.00 -> 82.7 mm
- net N$3: track 0.00 -> 50.8 mm
- net N$1: track 0.00 -> 35.3 mm
- net N$4: track 0.00 -> 34.8 mm
- net N$2: track 0.00 -> 19.6 mm
- net N$5: track 0.00 -> 9.90 mm
- added copper zone on layer 1, net GROUND
Other:
- board size 83.2 x 57.8 mm -> 160 x 100 mm
