File: light sensor basic.sch (EAGLE design)
At the start: 1 part

Commit message: Finished
Parts:
- added C2: 0.1uF, rcl:C-EUC1206
- added J1: UJ2-MIBH-G-SMT-TR, UJ2-MIBH-G-SMT-TR:UJ2-MIBH-G-SMT-TR
- added K<LED1: (no value), led:LEDCHIPLED_0805
- added Q1: (no value), semicon-smd-ipc:NPN-TRANSISTOR_SOT23
- added R1: 82, rcl:R-US_R1206
- added R2: TC33X-2-203E, TC33X-2-203E:TC33X-2-203E
- added R3: 150, rcl:R-US_R0805
- added TP1, TP2, TP3, TP4: (no value), rcl:R-US_R1206
- added U1: VCNT2020, VCNT2020:VCNT2020
Connections:
- new net GND: C2.1, J1.GND, J1.SHIELD, Q1.E, R2.CW, TP2.1, TP2.2, U1.CATHODE
- new net N$1: R1.2, U1.ANODE
- new net N$2: K<LED1.C, Q1.C
- new net N$3: R2.CCW, TP1.1, TP1.2, U1.EMITTER
- new net N$4: K<LED1.A, R3.1
- new net N$5: Q1.B, R2.W, TP3.1, TP3.2
- new net VCC: C2.2, J1.VCC, R1.1, R3.2, TP4.1, TP4.2, U1.COLLECTOR
